File: schematics/esp8266/esp8266.kicad_pcb (KiCad board)
At the start: 2 copper layers, 11 parts, among them P1 VCC, GND, P2 GPIO0->GND, P3 CONN_02X04, P4 RX, TX, U1 LM1084IS-3.3/NOPB

Commit message: Update eps8266 schematic
Parts:
- P3: value CONN_02X04 -> (none)
- P4: value RX, TX -> TX
- U1: value LM1084IS-3.3/NOPB -> (none)
Changed lines of the file:
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@@
   )
   (setup
-    (last_trace_width 0.8)
+    (last_trace_width 0.25)
     (user_trace_width 0.8)
     (trace_clearance 0.2)
@@
       (effects (font (size 1 1) (thickness 0.15)))
     )
-    (fp_text value "RX, TX" (at 15.24 -8.89) (layer F.Fab)
+    (fp_text value TX (at 15.24 -8.89) (layer F.Fab)
       (effects (font (size 1 1) (thickness 0.15)))
     )
@@
       (effects (font (size 1 1) (thickness 0.15)))
     )
-    (fp_text value LM1084IS-3.3/NOPB (at 0 3 90) (layer F.Fab)
+    (fp_text value "" (at 0 3 90) (layer F.Fab)
       (effects (font (size 1 1) (thickness 0.15)))
     )
@@
       (effects (font (size 1 1) (thickness 0.15)))
     )
-    (fp_text value CONN_02X04 (at 0 -3.1 270) (layer F.Fab)
+    (fp_text value "" (at 0 -3.1 270) (layer F.Fab)
       (effects (font (size 1 1) (thickness 0.15)))
     )
@@
   (segment (start 157.48 139.7) (end 157.48 144.78) (width 0.8) (layer F.Cu) (net 8))
   (segment (start 154.94 133.35) (end 154.94 137.16) (width 0.8) (layer F.Cu) (net 9))
-  (segment (start 154.94 130.81) (end 157.48 130.81) (width 0.8) (layer F.Cu) (net 10) (status C00000))
+  (segment (start 154.94 130.81) (end 157.48 130.81) (width 0.8) (layer F.Cu) (net 10))
   (segment (start 157.48 127) (end 157.48 130.81) (width 0.8) (layer F.Cu) (net 10))
   (segment (start 154.94 130.81) (end 153.67 130.81) (width 0.8) (layer F.Cu) (net 10))
