File: schematics/espDebug/espDebug.kicad_pcb (KiCad board)
At the start: 2 copper layers, 12 parts, among them P1 RAW, P2 3V3, P3 RX/TX, U1 SPX2920T-3.3, U2 ESP-201, U3 ESP8266, U4 button

Commit message: Update bugDebug schematic
Parts:
- moved P1 3.81 mm to (132.1, 85.1)
- moved P2 3.81 mm to (142.2, 87.6)
- moved P3 3.81 mm to (144.8, 92.7)
- moved U1 3.81 mm to (142.2, 82.5)
- moved U4 3.81 mm to (132.1, 92.7)
- moved R4 1.27 mm to (144.8, 115.6)
- moved R3 1.27 mm to (147.3, 108.0)
Routing:
- net Net-(D1-Pad1): track 110.5 -> 118.1 mm
- net Net-(U2-Pad5): track 38.1 -> 41.9 mm
- net Net-(P3-Pad2): track 23.9 -> 27.7 mm
- net Net-(P3-Pad1): track 30.0 -> 33.9 mm
- net Net-(P2-Pad1): track 41.7 -> 44.2 mm
- net Net-(R4-Pad1): track 19.6 -> 21.9 mm
- net Net-(R3-Pad2): track 12.7 -> 14.5 mm

Commit message: SCHMATIC: Update espDebug
Parts:
- added D2: LED, LEDs:LED-3MM, F.Cu at (127.0, 116.8)
- added R5: 1k, Resistors_ThroughHole:Resistor_Horizontal_RM7mm, F.Cu at (127.0, 111.8)
- moved D1 2.84 mm to (130.8, 116.8), turned to 90 degrees
- moved R1 1.27 mm to (130.8, 111.8)
Routing:
- net Net-(D1-Pad1): track 118.1 -> 201.3 mm
- net Net-(P3-Pad2): track 27.7 -> 85.1 mm
- net Net-(P2-Pad1): track 44.2 -> 65.8 mm
- net Net-(R5-Pad2): track 41.9 -> 51.3 mm
- net Net-(D2-Pad2): track 0.00 -> 2.54 mm
- net Net-(R1-Pad2): track 43.2 -> 44.4 mm
- net Net-(D1-Pad2): track 2.54 -> 3.17 mm
