File: schematics/matherboard/matherboard.kicad_pcb (KiCad board)
At the start: 2 copper layers, 12 parts, among them J1 RJ12, P1 VCC/GND, P4 CONN_01X05, U2 button, U3 STAB3.3, U4 ESP8266

Commit message: Schematic
Parts:
- removed U2: button, bugs:button
- added J2: RJ12, Connect:RJ12_E, F.Cu at (175.3, 83.8)
- added J3: RJ12, Connect:RJ12_E, F.Cu at (175.3, 124.5)
- added P2: CONN_01X02, Pin_Headers:Pin_Header_Straight_1x02, F.Cu at (129.5, 91.4)
- added P3: CONN_01X02, Pin_Headers:Pin_Header_Straight_1x02, F.Cu at (157.5, 99.1)
- added P5: CONN_01X05, Pin_Headers:Pin_Header_Straight_1x05, F.Cu at (162.6, 124.5)
- added P6: CONN_01X02, Pin_Headers:Pin_Header_Straight_1x02, F.Cu at (175.3, 109.2)
- P4: value CONN_01X05 -> CONN_01X02; footprint Pin_Headers:Pin_Header_Straight_1x05 -> Pin_Headers:Pin_Header_Straight_1x02
- R2, R4: footprint Resistors_ThroughHole:Resistor_Horizontal_RM7mm -> w_pth_resistors:rc03_vert
- moved P4 45.0 mm to (175.3, 99.1)
- moved J1 35.9 mm to (157.5, 83.8), turned to 180 degrees
- moved U3 31.8 mm to (132.1, 96.5), turned to 0 degrees
- moved D3 31.4 mm to (129.5, 111.8), turned to 0 degrees
- moved D2 16.9 mm to (129.5, 104.1)
- moved P1 15.5 mm to (129.5, 83.8), turned to 90 degrees
- moved R3 12.0 mm to (139.7, 104.1)
- moved R4 12.0 mm to (139.7, 86.4)
- moved R1 12.0 mm to (142.2, 104.1)
- moved R2 12.0 mm to (142.2, 86.4)
- moved U4 12.0 mm to (142.2, 94.0)
Connections:
- P4 pad 1: Net-(D2-Pad1) -> Net-(J2-Pad4)
- P4 pad 2: Net-(J1-Pad5) -> Net-(P3-Pad2)
- U3 pad 1: Net-(J1-Pad1) -> Net-(J1-Pad5)
- U4 pad 4: Net-(J1-Pad3) -> Net-(J1-Pad2)
- U4 pad 8: Net-(J1-Pad4) -> Net-(J1-Pad1)
Routing:
- net Net-(J1-Pad3): track 113.9 -> 0.00 mm
- net Net-(J1-Pad2): track 8.88 -> 113.7 mm
- net Net-(J1-Pad1): track 65.9 -> 170.6 mm
- net Net-(J1-Pad5): track 24.7 -> 120.5 mm
- net Net-(P3-Pad2): track 0.00 -> 58.0 mm
- net Net-(J1-Pad4): track 38.2 -> 6.56 mm
- net Net-(P1-Pad1): track 20.9 -> 5.08 mm
- net Net-(D3-Pad2): track 2.54 -> 14.8 mm
- net Net-(J3-Pad4): track 0.00 -> 6.56 mm
- net Net-(J2-Pad4): track 0.00 -> 6.56 mm
- net Net-(R2-Pad2): track 27.2 -> 20.8 mm
- net Net-(D2-Pad2): track 2.54 -> 7.62 mm
- net Net-(R4-Pad1): track 5.08 -> 3.81 mm
- net Net-(R2-Pad1): track 5.08 -> 3.81 mm
- net Net-(D2-Pad1): track 156.7 -> 155.9 mm
