File: schematics/raceSonar/raceSonar.sch (KiCad schematic (older format))
At the start: 13 parts, among them P1 CONN_01X08, P10 5V, P11 OUT1, P12 OUT2, P2 CONN_02X04, P4 CONN_02X07, P5 CONN_01X10, P6 CONTROL1, P7 CONTROL2, P8 35V, P9 GND, U1 Arduino_Mini, U2 L293D

Commit message: Schematic
Connections:
- net at P4.13 (P13), U1.10 (VCC): now also P4.1 (P1), P4.11 (P11), P4.3 (P3), P4.5 (P5), P4.7 (P7), P4.9 (P9)
- net at P2.7 (P7), U1.7 (RAW): now also P2.1 (P1), P2.3 (P3), P2.5 (P5)
- net at P2.2 (P2), P4.2 (P2), U1.8 (GND): now also P2.4 (P4), P2.6 (P6), P2.8 (P8), P4.10 (P10), P4.12 (P12), P4.14 (P14), P4.4 (P4), P4.6 (P6), P4.8 (P8)
Changed lines of the file:
@@
 Wire Wire Line
 	8400 4450 8550 4450
+Wire Wire Line
+	3150 4850 3350 4850
+Wire Wire Line
+	3250 3700 4050 3700
+Wire Wire Line
+	3250 4650 3150 4650
+Wire Wire Line
+	3250 3450 3250 4650
+Wire Wire Line
+	3350 4850 3350 4450
+Wire Wire Line
+	3350 4450 3500 4450
+Wire Wire Line
+	3150 4150 3150 4550
+Connection ~ 3250 3700
+Wire Wire Line
+	2150 4150 3150 4150
+$Comp
+L CONN_02X04 P2
+U 1 1 573AE72D
+P 2450 3900
+F 0 "P2" H 2450 4150 50  0000 C CNN
+F 1 "CONN_02X04" H 2450 3650 50  0000 C CNN
+F 2 "Pin_Headers:Pin_Header_Straight_2x04" H 2450 2700 50  0001 C CNN
+F 3 "" H 2450 2700 50  0000 C CNN
+	1    2450 3900
+	1    0    0    -1
+$EndComp
+Wire Wire Line
+	3450 3850 3450 4450
+Wire Wire Line
+	3450 4350 3500 4350
+Connection ~ 3450 4450
+Wire Wire Line
+	3450 4250 3500 4250
+Connection ~ 3450 4350
+Wire Wire Line
+	3450 4150 3500 4150
+Connection ~ 3450 4250
+Wire Wire Line
+	3450 4050 3500 4050
+Connection ~ 3450 4150
+Wire Wire Line
+	3450 3950 3500 3950
+Connection ~ 3450 4050
+Wire Wire Line
+	3450 3850 3500 3850
+Connection ~ 3450 3950
 $Comp
 L CONN_02X07 P4
@@
 $EndComp
 Wire Wire Line
-	3150 4850 3350 4850
+	4050 3700 4050 4450
 Wire Wire Line
-	3250 3700 4000 3700
+	4050 3850 4000 3850
 Wire Wire Line
-	4000 3700 4000 3850
+	4050 3950 4000 3950
+Connection ~ 4050 3850
 Wire Wire Line
-	3250 4650 3150 4650
+	4050 4050 4000 4050
+Connection ~ 4050 3950
 Wire Wire Line
-	3250 3450 3250 4650
+	4050 4150 4000 4150
+Connection ~ 4050 4050
 Wire Wire Line
-	3350 4850 3350 4450
+	4050 4250 4000 4250
+Connection ~ 4050 4150
 Wire Wire Line
-	3350 4450 3500 4450
+	4050 4350 4000 4350
+Connection ~ 4050 4250
 Wire Wire Line
-	3150 4150 3150 4550
+	4050 4450 4000 4450
+Connection ~ 4050 4350
 Wire Wire Line
-	3250 3450 2700 3450
-Connection ~ 3250 3700
+	2150 3750 2150 4150
 Wire Wire Line
-	2200 4050 2200 4150
+	2150 4050 2200 4050
 Wire Wire Line
-	2200 4150 3150 4150
-$Comp
-L CONN_02X04 P2
-U 1 1 573AE72D
-P 2450 3900
-F 0 "P2" H 2450 4150 50  0000 C CNN
-F 1 "CONN_02X04" H 2450 3650 50  0000 C CNN
-F 2 "Pin_Headers:Pin_Header_Straight_2x04" H 2450 2700 50  0001 C CNN
-F 3 "" H 2450 2700 50  0000 C CNN
-	1    2450 3900
-	1    0    0    -1
-$EndComp
+	2200 3950 2150 3950
+Connection ~ 2150 4050
 Wire Wire Line
-	2700 3450 2700 3750
+	2200 3850 2150 3850
+Connection ~ 2150 3950
+Wire Wire Line
+	2200 3750 2150 3750
+Connection ~ 2150 3850
+Wire Wire Line
+	2700 3750 2750 3750
+Wire Wire Line
+	2750 3450 3250 3450
+Wire Wire Line
+	2750 3450 2750 4050
+Wire Wire Line
+	2750 3850 2700 3850
+Connection ~ 2750 3750
+Wire Wire Line
+	2750 3950 2700 3950
+Connection ~ 2750 3850
+Wire Wire Line
+	2750 4050 2700 4050
+Connection ~ 2750 3950
 $EndSCHEMATC
